File: hayabusa04.sch (KiCad schematic (older format))
At the start: 24 parts, among them SW1 SW_Push, U1 ATmega32U4-AU, Y1 16MHz

Commit message: updated pcb
Connections:
- net COL0: now also U1.29 (PB5)
- net COL1: now also U1.28 (PB4)
- net ROW0: now also U1.27 (PD7)
- net ROW1: now also U1.30 (PB6)
Changed lines of the file:
@@
 Text GLabel 5400 4000 0    50   Input ~ 0
 ROW1
+Text GLabel 3650 2700 2    50   Input ~ 0
+COL1
+Text GLabel 3650 2800 2    50   Input ~ 0
+COL0
+Text GLabel 3650 2900 2    50   Input ~ 0
+ROW1
+Text GLabel 3650 4200 2    50   Input ~ 0
+ROW0
 $EndSCHEMATC

Commit message: test
Parts:
- added R?: R_Small, symbol Device:R_Small
Changed lines of the file:
@@
 EESchema Schematic File Version 4
+LIBS:hayabusa04-cache
 EELAYER 30 0
 EELAYER END
@@
 Text GLabel 3650 4200 2    50   Input ~ 0
 ROW0
+$Comp
+L Device:R_Small R?
+U 1 1 634ADF57
+P 8100 2300
+F 0 "R?" H 8159 2346 50  0000 L CNN
+F 1 "R_Small" H 8159 2255 50  0000 L CNN
+F 2 "" H 8100 2300 50  0001 C CNN
+F 3 "~" H 8100 2300 50  0001 C CNN
+	1    8100 2300
+	1    0    0    -1
+$EndComp
 $EndSCHEMATC
