File: hayabusa04.kicad_sch (KiCad schematic)
At the start: 20 parts, among them SW1 SW_Push, SW2 MX_SW_HS, SW3 MX_SW_HS, SW4 MX_SW_HS, SW5 MX_SW_HS, U1 ATmega32U4-AU, Y1 16MHz

Commit message: routed usb c
Parts:
- removed USB1: Molex-0548190589, random-keyboard-parts:Molex-0548190589, symbol random-keyboard-parts:Molex-0548190589
- added J1: USB_C_Receptacle_USB2.0, Connector_USB:USB_C_Receptacle_HRO_TYPE-C-31-M-12, symbol Connector:USB_C_Receptacle_USB2.0
- added R5, R6: 5.1k, Resistor_SMD:R_0805_2012Metric, symbol Device:R_Small
- added U2: SRV05-4, Package_TO_SOT_SMD:SOT-23-6, symbol Power_Protection:SRV05-4
Connections:
- net VCC is gone; now on net +5V: F1.2
- net +5V: no longer F1.1
- net D+: now also J1.A6 (D+), J1.B6 (D+), U2.3 (IO2)
- net D-: now also J1.A7 (D-), J1.B7 (D-), U2.4 (IO3)
- net GND: now also J1.A1 (GND), J1.A12 (GND), J1.B1 (GND), J1.B12 (GND), J1.S1 (SHIELD), R5.1, R6.2, U2.2 (VN)
- new net CC1: J1.A5 (CC1), R5.2, U2.6 (IO4)
- new net CC2: J1.B5 (CC2), R6.1, U2.1 (IO1)
- new net ESD5V: F1.1, J1.A4 (VBUS), J1.A9 (VBUS), J1.B4 (VBUS), J1.B9 (VBUS), U2.5 (VP)
- no-connect marks 0 -> 24
Other:
- moved on the sheet: SW2, SW3, SW4, SW5
